Commit message: update

File: legged_gym/resources/robots/mybot_v2_1/urdf/mybot_v2_1.urdf (robot description, URDF)
Before this commit: robot mybot_v2_1, 18 links, 17 joints
Links:
- link FL_hip: geometry visual mesh filename=../meshes/FL_hip.STL
- link FR_hip: geometry visual mesh filename=../meshes/FR_hip.STL
- link RL_hip: geometry visual mesh filename=../meshes/RL_hip.STL
- link RR_hip: geometry visual mesh filename=../meshes/RR_hip.STL
Joints:
- removed joint FL_foot_joint
- removed joint FR_foot_joint
- removed joint RL_foot_joint
- removed joint RR_foot_joint
- added joint FL_foot_fixed: type fixed, parent FL_calf, child FL_foot, origin xyz=0 -0.00025 -0.22336 rpy=0 0 0, axis 0 0 0
- added joint FR_foot_fixed: type fixed, parent FR_calf, child FR_foot, origin xyz=0 0.00025000000001113 -0.223362537893242 rpy=0 0 0, axis 0 0 0
- added joint RL_foot_fixed: type fixed, parent RL_calf, child RL_foot, origin xyz=0 -0.000250000000010231 -0.223362537894357 rpy=0 0 0, axis 0 0 0
- added joint RR_foot_fixed: type fixed, parent RR_calf, child RR_foot, origin xyz=0 0.000250000000008521 -0.223362537894357 rpy=0 0 0, axis 0 0 0
